Commit message: rl code for y4a -- deploy version

File: resources/robots/y4a/urdf/y4aurdf20250827.urdf (robot description, URDF)
Before this commit: robot y4aurdf20250827, 9 links, 8 joints
Joints:
- joint left_wheel_joint: limit lower=-10000000 upper=10000000 effort=192 velocity=17.017 -> lower=-10000000 upper=10000000 effort=60 velocity=15.603
- joint right_wheel_joint: limit lower=-10000000 upper=10000000 effort=192 velocity=17.017 -> lower=-10000000 upper=10000000 effort=60 velocity=15.603

File: sim/model/y4a/urdf/y4aurdf20250827.urdf (robot description, URDF)
Before this commit: robot y4aurdf20250827, 9 links, 8 joints
Joints:
- joint left_wheel_joint: limit lower=-10000000 upper=10000000 effort=192 velocity=17.017 -> lower=-10000000 upper=10000000 effort=60 velocity=15.603
- joint right_wheel_joint: limit lower=-10000000 upper=10000000 effort=192 velocity=17.017 -> lower=-10000000 upper=10000000 effort=60 velocity=15.603
