Commit message: code stashed

File: resources/robots/y4b/urdf/y4burdf20260114_bk.urdf (robot description, URDF)
Before this commit: robot y4burdf20260114, 9 links, 8 joints
Links:
- link base_link: mass 9.7803 -> 9.3994; geometry collision mesh filename=package://y4burdf20260114/meshes/base_link.STL; visual mesh filename=package://y4burdf20260114/meshes/base_link.STL
- link left_hip_pitch_link: geometry collision mesh filename=package://y4burdf20260114/meshes/left_hip_pitch_link.STL; visual mesh filename=package://y4burdf20260114/meshes/left_hip_pitch_link.STL
- link left_hip_roll_link: geometry collision mesh filename=package://y4burdf20260114/meshes/left_hip_roll_link.STL; visual mesh filename=package://y4burdf20260114/meshes/left_hip_roll_link.STL
- link left_knee_link: geometry collision mesh filename=package://y4burdf20260114/meshes/left_knee_link.STL; visual mesh filename=package://y4burdf20260114/meshes/left_knee_link.STL
- link left_wheel_link: mass 0.94045 -> 1.432; geometry collision mesh filename=package://y4burdf20260114/meshes/left_wheel_link.STL; visual mesh filename=package://y4burdf20260114/meshes/left_wheel_link.STL
- link right_hip_pitch_link: geometry collision mesh filename=package://y4burdf20260114/meshes/right_hip_pitch_link.STL; visual mesh filename=package://y4burdf20260114/meshes/right_hip_pitch_link.STL
- link right_hip_roll_link: geometry collision mesh filename=package://y4burdf20260114/meshes/right_hip_roll_link.STL; visual mesh filename=package://y4burdf20260114/meshes/right_hip_roll_link.STL
- link right_knee_link: geometry collision mesh filename=package://y4burdf20260114/meshes/right_knee_link.STL; visual mesh filename=package://y4burdf20260114/meshes/right_knee_link.STL
- link right_wheel_link: mass 0.94045 -> 1.432; geometry collision mesh filename=package://y4burdf20260114/meshes/right_wheel_link.STL; visual mesh filename=package://y4burdf20260114/meshes/right_wheel_link.STL

File: sim/model/y4b/urdf/y4burdf20260114.urdf (robot description, URDF)
Before this commit: robot y4burdf20260114, 9 links, 8 joints
Links:
- link base_link: mass 9.3994 -> 9.7803
- link left_wheel_link: mass 1.432 -> 0.94045
- link right_wheel_link: mass 1.432 -> 0.94045
